Commit message: start of hardware interface

File: description/ros2_control/robot.ros2_control.xacro (robot description, xacro)
@@ -5,15 +5,16 @@
       <hardware>
         <plugin>odrive_ros2_control_example/RobotHardwareInterface</plugin>
-        <param name="debug">true</param>
+        <param name="debug">1</param>
       </hardware>
       <joint name="arm">
+        <!-- Parameters -->
+        <param name="node_id">0</param>
+        <param name="reduction_ratio">1</param>
+        <param name="velocity_limit">10</param>
+        <param name="effort_limit">5</param>
         <!-- Command Interfaces (Input) -->
         <command_interface name="position" data_type="double"/>
         <command_interface name="velocity" data_type="double"/>
-        <command_interface name="torque" data_type="double"/>
-        <command_interface name="position_lower_limit" data_type="double"/>
-        <command_interface name="position_upper_limit" data_type="double"/>
-        <command_interface name="velocity_limit" data_type="double"/>
-        <command_interface name="torque_limit" data_type="double"/>
+        <command_interface name="effort" data_type="double"/>
         <!-- State Interfaces (Output) -->
         <state_interface name="position" data_type="double">
@@ -23,5 +24,5 @@
           <param name="initial_value">0.0</param>
         </state_interface>
-        <state_interface name="torque" data_type="double">
+        <state_interface name="effort" data_type="double">
           <param name="initial_value">0.0</param>
         </state_interface>

File: description/urdf/robot.urdf.xacro (robot description, xacro)
@@ -35,5 +35,5 @@
     <child link="body"/>
   </joint>
-  <joint name="body_to_arm" type="continuous">
+  <joint name="arm" type="continuous">
     <origin rpy="0 0 0" xyz="0 -0.075 0"/>
     <parent link="body"/>
